File: EDA/quack_connectors.kicad_sch (KiCad schematic)
At the start: 32 parts, among them J1 DIN-4, J2 DB9_Male, J3 FTDI, Q1 SI2301CDS-T1-GE3, SW1 SW_DIP_x03, U2 SN74LVC2T45YZP, U4 SN74LVC4245APWR

Commit message: EDA lib: updated Mini DIN 4 connector
Parts:
- J1: footprint Quack_MDIN4:57491811 -> Quack_MDIN4:5749181-1
Changed lines of the file:
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@@
 			)
 		)
-		(property "Footprint" "Quack_MDIN4:57491811"
+		(property "Footprint" "Quack_MDIN4:5749181-1"
 			(at 247.65 44.45 0)
 			(effects
